Commit message: first commit

File: description/robot_core.xacro (robot description, xacro)
@@ -37,7 +37,7 @@
             </geometry>
         </collision>
-        <xacro:intertial_box mass = "0.5" x = "0.3" y = "0.3" z = "0.15">
-            <origin xyz = "0.15 0 0.075"/>
-        </xacro:intertial_box>
+        <xacro:inertial_box mass = "0.5" x = "0.3" y = "0.3" z = "0.15">
+            <origin xyz = "0.15 0 0.075" rpy = "0 0 0" />
+        </xacro:inertial_box>
     </link>
     <!-- LEFT WHEEL LINK-->
@@ -60,6 +60,6 @@
             </geometry>
         </collision>
-        <xacro:inertial_cylinder mass = "0.1" length = " 0.04" radius = " 0.05">
-            <origin xyz = "0 0 0" rpy = "0 0 0 "/>
+        <xacro:inertial_cylinder mass = "0.1" length = "0.04" radius = "0.05">
+            <origin xyz = "0 0 0" rpy = "0 0 0" />
         </xacro:inertial_cylinder>
     </link>
@@ -83,6 +83,6 @@
             </geometry>
         </collision>
-        <xacro:inertial_cylinder mass = "0.1" length = " 0.04" radius = " 0.05">
-            <origin xyz = "0 0 0" rpy = "0 0 0 "/>
+        <xacro:inertial_cylinder mass = "0.1" length = "0.04" radius = "0.05">
+            <origin xyz = "0 0 0" rpy = "0 0 0" />
         </xacro:inertial_cylinder>
     </link>
@@ -105,7 +105,7 @@
             </geometry>
         </collision>
-        <xacro:intertial_sphere mass = "0.1" radius = "0.05">
+        <xacro:inertial_sphere mass = "0.1" radius = "0.05">
             <origin xyz = "0 0 0" rpy = "0 0 0"/>
-        </xacro:intertial_sphere>
+        </xacro:inertial_sphere>
     </link>
 </robot>
