Commit message: new_launch

File: description/ros2_control.xacro (robot description, xacro)
@@ -1,10 +1,11 @@
 <?xml version="1.0"?>
 <robot xmlns:xacro="http://www.ros.org/wiki/xacro"  name="robot">
-  <ros2_control name="GazeboSystem" type="system">
+  <ros2_control name="GazeboSymSystem" type="system">
     <hardware>
         <plugin>
             gazebo_ros2_control/GazeboSystem
         </plugin>
-        <joint name="left_wheel_joint">
+    </hardware>
+    <joint name="left_wheel_joint">
             <command_interface name="velocity">
                 <param name="min">-10</param>
@@ -13,6 +14,6 @@
             <state_interface name="velocity"/>
             <state_interface name="position"/>
-        </joint>
-        <joint name="right_wheel_joint">
+    </joint>
+    <joint name="right_wheel_joint">
             <command_interface name="velocity">
                 <param name="min">-10</param>
@@ -21,6 +22,5 @@
             <state_interface name="velocity"/>
             <state_interface name="position"/>
-        </joint>
-    </hardware>
+    </joint>
   </ros2_control>
   <gazebo>
